Commit message: Nov 29 Add FabMJCFForwardKinematics, providing fk directly from MJCF/XML

File: mjpc/tasks/planar_robot/planar_2dof.urdf (robot description, URDF)
Before this commit: robot planar_2dof, 5 links, 4 joints
Links:
- removed link link3
- added link tip, mass 0.0001; collision sphere radius=0.1; visual sphere radius=0.1
Joints:
- joint joint3: child link3 -> tip
